Commit message: update slip control

File: slip/urdf/slip.urdf (robot description, URDF)
Before this commit: robot slip, 4 links, 3 joints
Joints:
- joint joint3: limit lower=-0.1 upper=0.5 effort=3000.0 velocity=10 -> lower=-0.1 upper=0.7 effort=3000.0 velocity=10

Commit message: update energy control

File: slip/urdf/slip.urdf (robot description, URDF)
Before this commit: robot slip, 4 links, 3 joints
Links:
- link link1: mass 0.002 -> 0.46057
